File: pcb/micro-sci.sch (KiCad schematic (older format))
At the start: 46 parts, among them J1 ISP, U1 ATmega328P-PU, X1 12 MHz

Commit message: Update schematic
Connections:
- net +5V: now also J1.1 (Pin_1)
- net C1: now also U1.14 (PB0)
- net C2: now also U1.16 (PB2)
- net GND: now also J1.2 (Pin_2)
- net R1: now also U1.23 (PC0)
- net R2: now also U1.24 (PC1)
- net R3: now also U1.25 (PC2)
- net R4: now also U1.26 (PC3)
- net R5: now also U1.27 (PC4)
- net R6: now also U1.28 (PC5)
- net R7: now also U1.2 (PD0)
- net R8: now also U1.3 (PD1)
- net RESET: now reaches U1.1 (~RESET~/PC6)
- net RESET: now also J1.6 (Pin_6)
- net at U1.11 (PD5): now also DS1.12 (D5)
- net at U1.12 (PD6): now also DS1.13 (D6)
- net at U1.13 (PD7): now also DS1.14 (D7)
- net at U1.15 (PB1): now also DS1.16 (LED(-))
- net MOSI: now reaches U1.17 (PB3)
- net MOSI: now also J1.4 (Pin_4)
- net MISO: now reaches U1.18 (PB4)
- net MISO: now also J1.5 (Pin_5)
- net SCK: now reaches U1.19 (PB5)
- net SCK: now also J1.3 (Pin_3)
- net at U1.4 (PD2): now also DS1.6 (E)
- net at U1.5 (PD3): now also DS1.4 (RS)
- net at U1.6 (PD4): now also DS1.11 (D4)
Changed lines of the file:
@@
 EESchema Schematic File Version 4
+LIBS:micro-sci-cache
 EELAYER 26 0
 EELAYER END
@@
 Sheet 1 1
 Title "MicroSci"
-Date "2020-06-07"
-Rev "0.9"
+Date "2020-06-09"
+Rev "1.0"
 Comp "Paweł Kania"
 Comment1 ""
@@
 Comment4 ""
 $EndDescr
-$Comp
-L MCU_Microchip_ATmega:ATmega328P-PU U1
-U 1 1 5EDD3B9E
-P 2950 3300
-F 0 "U1" H 2309 3346 50  0000 R CNN
-F 1 "ATmega328P-PU" H 2309 3255 50  0000 R CNN
-F 2 "Package_DIP:DIP-28_W7.62mm" H 2950 3300 50  0001 C CIN
-F 3 "http://ww1.microchip.com/downloads/en/DeviceDoc/ATmega328_P%20AVR%20MCU%20with%20picoPower%20Technology%20Data%20Sheet%2040001984A.pdf" H 2950 3300 50  0001 C CNN
-	1    2950 3300
-	1    0    0    -1
-$EndComp
 $Comp
 L Device:C C2
@@
 Wire Wire Line
 	4100 4950 5250 4950
+Wire Wire Line
+	4850 4250 4850 4500
+Wire Wire Line
+	4850 4500 3550 4500
+Wire Wire Line
+	4850 4150 4750 4150
+Wire Wire Line
+	4750 4150 4750 4400
+Wire Wire Line
+	4750 4400 3550 4400
+Wire Wire Line
+	4850 4050 4650 4050
+Wire Wire Line
+	4650 4050 4650 4300
+Wire Wire Line
+	4650 4300 3550 4300
+Wire Wire Line
+	4850 3950 4550 3950
+Wire Wire Line
+	4550 3950 4550 4200
+Wire Wire Line
+	4550 4200 3550 4200
+Wire Wire Line
+	4850 3250 4750 3250
+Wire Wire Line
+	4750 3250 4750 3850
+Wire Wire Line
+	4750 3850 4450 3850
+Wire Wire Line
+	4450 3850 4450 4100
+Wire Wire Line
+	4450 4100 3550 4100
+Wire Wire Line
+	4850 3050 4650 3050
+Wire Wire Line
+	4650 3050 4650 3750
+Wire Wire Line
+	4650 3750 4350 3750
+Wire Wire Line
+	4350 3750 4350 4000
+Wire Wire Line
+	4350 4000 3550 4000
+Text GLabel 4950 1650 0    50   Output ~ 0
+RESET
+$Comp
+L power:+5V #PWR?
+U 1 1 5EE54026
+P 4800 1000
+F 0 "#PWR?" H 4800 850 50  0001 C CNN
+F 1 "+5V" H 4815 1173 50  0000 C CNN
+F 2 "" H 4800 1000 50  0001 C CNN
+F 3 "" H 4800 1000 50  0001 C CNN
+	1    4800 1000
+	0    -1   -1   0
+$EndComp
+$Comp
+L power:GND #PWR?
+U 1 1 5EE5EAD3
+P 4800 1150
+F 0 "#PWR?" H 4800 900 50  0001 C CNN
+F 1 "GND" H 4805 977 50  0000 C CNN
+F 2 "" H 4800 1150 50  0001 C CNN
+F 3 "" H 4800 1150 50  0001 C CNN
+	1    4800 1150
+	0    1    1    0
+$EndComp
+Wire Wire Line
+	4950 1150 4950 1000
+Wire Wire Line
+	4950 1000 4800 1000
+Wire Wire Line
+	4950 1250 4800 1250
+Wire Wire Line
+	4800 1250 4800 1150
+Text GLabel 3550 3600 2    50   Input ~ 0
+RESET
+Wire Wire Line
+	3550 2200 5900 2200
+Wire Wire Line
+	5900 2200 5900 3450
+Wire Wire Line
+	5900 3450 5650 3450
+$Comp
+L MCU_Microchip_ATmega:ATmega328P-PU U1
+U 1 1 5EDD3B9E
+P 2950 3300
+F 0 "U1" H 2309 3346 50  0000 R CNN
+F 1 "ATmega328P-PU" H 2309 3255 50  0000 R CNN
+F 2 "Package_DIP:DIP-28_W7.62mm" H 2950 3300 50  0001 C CIN
+F 3 "http://ww1.microchip.com/downloads/en/DeviceDoc/ATmega328_P%20AVR%20MCU%20with%20picoPower%20Technology%20Data%20Sheet%2040001984A.pdf" H 2950 3300 50  0001 C CNN
+	1    2950 3300
+	1    0    0    -1
+$EndComp
+Wire Wire Line
+	3550 2400 4100 2400
+Wire Wire Line
+	3550 2500 4200 2500
+Wire Wire Line
+	3750 2600 3750 2250
+Wire Wire Line
+	3750 2250 4000 2250
+Wire Wire Line
+	3550 2600 3750 2600
+Text GLabel 3550 2100 2    50   BiDi ~ 0
+C1
+Text GLabel 3550 2300 2    50   BiDi ~ 0
+C2
+Text GLabel 3550 3000 2    50   BiDi ~ 0
+R1
+Text GLabel 3550 3100 2    50   BiDi ~ 0
+R2
+Text GLabel 3550 3200 2    50   BiDi ~ 0
+R3
+Text GLabel 3550 3300 2    50   BiDi ~ 0
+R4
+Text GLabel 3550 3400 2    50   BiDi ~ 0
+R5
+Text GLabel 3550 3500 2    50   BiDi ~ 0
+R6
+Text GLabel 3550 3800 2    50   BiDi ~ 0
+R7
+Text GLabel 3550 3900 2    50   BiDi ~ 0
+R8
+Wire Wire Line
+	4000 1350 4950 1350
+Wire Wire Line
+	4000 1350 4000 2250
+Wire Wire Line
+	4100 1450 4950 1450
+Wire Wire Line
+	4100 1450 4100 2400
+Wire Wire Line
+	4200 1550 4950 1550
+Wire Wire Line
+	4200 1550 4200 2500
+Text Label 4950 1350 2    50   ~ 0
+SCK
+Text Label 4950 1450 2    50   ~ 0
+MOSI
+Text Label 4950 1550 2    50   ~ 0
+MISO
 $EndSCHEMATC
